Commit message: panda arm spatula

File: panda/panda_arm_spatula.urdf (robot description, URDF)
Before this commit: robot panda, 9 links, 8 joints
Links:
- link end-effector: geometry collision box size=0.2286 0.2286 0.002; visual box size=0.2286 0.2286 0.002

Commit message: new end effector

File: panda/panda_arm_spatula.urdf (robot description, URDF)
Before this commit: robot panda, 9 links, 8 joints
Links:
- link end-effector: geometry collision box size=0.195 0.195 0.003; visual box size=0.195 0.195 0.003
Joints:
- joint joint_ee: origin xyz=0 0 0.14 rpy=0 0 0 -> xyz=0 0 0.14 rpy=0 0 -1.57

Commit message: urdf

File: panda/panda_arm_spatula.urdf (robot description, URDF)
Before this commit: robot panda, 9 links, 8 joints
Links:
- added link intermediate-end-effector, mass 0.1
- link end-effector: geometry visual box size=0.2119 0.2032 0.0032
Joints:
- added joint joint_ee_2: type fixed, parent intermediate-end-effector, child end-effector, origin xyz=-0.0963 0 0 rpy=0 3.925 0
- joint joint_ee: child end-effector -> intermediate-end-effector; origin xyz=0 0 0.14 rpy=0 0 -1.57 -> xyz=0 0 0.2794 rpy=0 0 -0.785

Commit message: sharing code...

File: panda/panda_arm_spatula.urdf (robot description, URDF)
Before this commit: robot panda, 9 links, 8 joints
Links:
- added link intermediate-end-effector, mass 0.1
- link end-effector: geometry collision box size=0.2119 0.2032 0.0032; visual box size=0.2119 0.2032 0.0032
Joints:
- added joint joint_ee_2: type fixed, parent intermediate-end-effector, child end-effector, origin xyz=-0.0963 0 0 rpy=0 3.925 0
- joint joint_ee: child end-effector -> intermediate-end-effector; origin xyz=0 0 0.14 rpy=0 0 -1.57 -> xyz=0 0 0.2794 rpy=0 0 -0.785
